File: hardware/LCD Module/LCD Module/LCD Module.kicad_pcb (KiCad board)
At the start: 2 copper layers, 53.3 x 32.2 mm, 11 parts, among them J1 Conn_02x04_Counter_Clockwise

Commit message: Working on v2 of HW
Changed lines of the file:
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@@
       (outputformat 1)
       (mirror false)
-      (drillshape 1)
+      (drillshape 0)
       (scaleselection 1)
-      (outputdirectory "")
+      (outputdirectory "Gerbers/")
     )
   )
@@
     (fp_line (start 1.6 0.8) (end 1.6 -0.8)
       (stroke (width 0.1) (type solid)) (layer "B.Fab"))
-    (pad "1" smd roundrect (at -1.5625 0 270) (size 1.325 1.8) (layers "B.Cu" "B.Paste" "B.Mask") (roundrect_rratio 0.188679)
+    (pad "1" smd roundrect (at -1.5625 0 270) (size 1.325 1.8) (layers "B.Cu" "B.Paste" "B.Mask") (roundrect_rratio 0.1886792453)
       (net 6 "Net-(LCDScreen1-C2-)") (pintype "passive"))
-    (pad "2" smd roundrect (at 1.5625 0 270) (size 1.325 1.8) (layers "B.Cu" "B.Paste" "B.Mask") (roundrect_rratio 0.188679)
+    (pad "2" smd roundrect (at 1.5625 0 270) (size 1.325 1.8) (layers "B.Cu" "B.Paste" "B.Mask") (roundrect_rratio 0.1886792453)
       (net 7 "Net-(LCDScreen1-C2+)") (pintype "passive"))
     (model "${KICAD6_3DMODEL_DIR}/Capacitor_SMD.3dshapes/C_1206_3216Metric.wrl"
@@
     (fp_line (start 1.6 0.8) (end 1.6 -0.8)
       (stroke (width 0.1) (type solid)) (layer "B.Fab"))
-    (pad "1" smd roundrect (at -1.5625 0 270) (size 1.325 1.8) (layers "B.Cu" "B.Paste" "B.Mask") (roundrect_rratio 0.188679)
+    (pad "1" smd roundrect (at -1.5625 0 270) (size 1.325 1.8) (layers "B.Cu" "B.Paste" "B.Mask") (roundrect_rratio 0.1886792453)
       (net 1 "GND") (pintype "passive"))
-    (pad "2" smd roundrect (at 1.5625 0 270) (size 1.325 1.8) (layers "B.Cu" "B.Paste" "B.Mask") (roundrect_rratio 0.188679)
+    (pad "2" smd roundrect (at 1.5625 0 270) (size 1.325 1.8) (layers "B.Cu" "B.Paste" "B.Mask") (roundrect_rratio 0.1886792453)
       (net 8 "Net-(LCDScreen1-V2)") (pintype "passive"))
     (model "${KICAD6_3DMODEL_DIR}/Capacitor_SMD.3dshapes/C_1206_3216Metric.wrl"
@@
     (fp_line (start 1.6 0.8) (end 1.6 -0.8)
       (stroke (width 0.1) (type solid)) (layer "B.Fab"))
-    (pad "1" smd roundrect (at -1.5625 0 270) (size 1.325 1.8) (layers "B.Cu" "B.Paste" "B.Mask") (roundrect_rratio 0.188679)
+    (pad "1" smd roundrect (at -1.5625 0 270) (size 1.325 1.8) (layers "B.Cu" "B.Paste" "B.Mask") (roundrect_rratio 0.1886792453)
       (net 1 "GND") (pintype "passive"))
-    (pad "2" smd roundrect (at 1.5625 0 270) (size 1.325 1.8) (layers "B.Cu" "B.Paste" "B.Mask") (roundrect_rratio 0.188679)
+    (pad "2" smd roundrect (at 1.5625 0 270) (size 1.325 1.8) (layers "B.Cu" "B.Paste" "B.Mask") (roundrect_rratio 0.1886792453)
       (net 11 "Net-(LCDScreen1-V1)") (pintype "passive"))
     (model "${KICAD6_3DMODEL_DIR}/Capacitor_SMD.3dshapes/C_1206_3216Metric.wrl"
@@
     (fp_line (start 1.6 0.8) (end 1.6 -0.8)
       (stroke (width 0.1) (type solid)) (layer "B.Fab"))
-    (pad "1" smd roundrect (at -1.5625 0 270) (size 1.325 1.8) (layers "B.Cu" "B.Paste" "B.Mask") (roundrect_rratio 0.188679)
+    (pad "1" smd roundrect (at -1.5625 0 270) (size 1.325 1.8) (layers "B.Cu" "B.Paste" "B.Mask") (roundrect_rratio 0.1886792453)
       (net 9 "Net-(LCDScreen1-C1+)") (pintype "passive"))
-    (pad "2" smd roundrect (at 1.5625 0 270) (size 1.325 1.8) (layers "B.Cu" "B.Paste" "B.Mask") (roundrect_rratio 0.188679)
+    (pad "2" smd roundrect (at 1.5625 0 270) (size 1.325 1.8) (layers "B.Cu" "B.Paste" "B.Mask") (roundrect_rratio 0.1886792453)
       (net 10 "Net-(LCDScreen1-C1-)") (pintype "passive"))
     (model "${KICAD6_3DMODEL_DIR}/Capacitor_SMD.3dshapes/C_1206_3216Metric.wrl"
@@
     (fp_line (start 1.6 0.8) (end 1.6 -0.8)
       (stroke (width 0.1) (type solid)) (layer "B.Fab"))
-    (pad "1" smd roundrect (at -1.5625 0 270) (size 1.325 1.8) (layers "B.Cu" "B.Paste" "B.Mask") (roundrect_rratio 0.188679)
+    (pad "1" smd roundrect (at -1.5625 0 270) (size 1.325 1.8) (layers "B.Cu" "B.Paste" "B.Mask") (roundrect_rratio 0.1886792453)
       (net 1 "GND") (pintype "passive"))
-    (pad "2" smd roundrect (at 1.5625 0 270) (size 1.325 1.8) (layers "B.Cu" "B.Paste" "B.Mask") (roundrect_rratio 0.188679)
+    (pad "2" smd roundrect (at 1.5625 0 270) (size 1.325 1.8) (layers "B.Cu" "B.Paste" "B.Mask") (roundrect_rratio 0.1886792453)
       (net 2 "Net-(LCDScreen1-V0)") (pintype "passive"))
     (model "${KICAD6_3DMODEL_DIR}/Capacitor_SMD.3dshapes/C_1206_3216Metric.wrl"
@@
     (fp_line (start 1.6 0.8) (end 1.6 -0.8)
       (stroke (width 0.1) (type solid)) (layer "B.Fab"))
-    (pad "1" smd roundrect (at -1.5625 0 270) (size 1.325 1.8) (layers "B.Cu" "B.Paste" "B.Mask") (roundrect_rratio 0.188679)
+    (pad "1" smd roundrect (at -1.5625 0 270) (size 1.325 1.8) (layers "B.Cu" "B.Paste" "B.Mask") (roundrect_rratio 0.1886792453)
       (net 1 "GND") (pintype "passive"))
-    (pad "2" smd roundrect (at 1.5625 0 270) (size 1.325 1.8) (layers "B.Cu" "B.Paste" "B.Mask") (roundrect_rratio 0.188679)
+    (pad "2" smd roundrect (at 1.5625 0 270) (size 1.325 1.8) (layers "B.Cu" "B.Paste" "B.Mask") (roundrect_rratio 0.1886792453)
       (net 3 "Net-(LCDScreen1-V4)") (pintype "passive"))
     (model "${KICAD6_3DMODEL_DIR}/Capacitor_SMD.3dshapes/C_1206_3216Metric.wrl"
@@
     (fp_line (start 1.6 0.8) (end 1.6 -0.8)
       (stroke (width 0.1) (type solid)) (layer "B.Fab"))
-    (pad "1" smd roundrect (at -1.5625 0 270) (size 1.325 1.8) (layers "B.Cu" "B.Paste" "B.Mask") (roundrect_rratio 0.188679)
+    (pad "1" smd roundrect (at -1.5625 0 270) (size 1.325 1.8) (layers "B.Cu" "B.Paste" "B.Mask") (roundrect_rratio 0.1886792453)
       (net 1 "GND") (pintype "passive"))
-    (pad "2" smd roundrect (at 1.5625 0 270) (size 1.325 1.8) (layers "B.Cu" "B.Paste" "B.Mask") (roundrect_rratio 0.188679)
+    (pad "2" smd roundrect (at 1.5625 0 270) (size 1.325 1.8) (layers "B.Cu" "B.Paste" "B.Mask") (roundrect_rratio 0.1886792453)
       (net 5 "Net-(LCDScreen1-V3)") (pintype "passive"))
     (model "${KICAD6_3DMODEL_DIR}/Capacitor_SMD.3dshapes/C_1206_3216Metric.wrl"
@@
     (fp_line (start 1.6 0.8) (end 1.6 -0.8)
       (stroke (width 0.1) (type solid)) (layer "B.Fab"))
-    (pad "1" smd roundrect (at -1.5625 0 270) (size 1.325 1.8) (layers "B.Cu" "B.Paste" "B.Mask") (roundrect_rratio 0.188679)
+    (pad "1" smd roundrect (at -1.5625 0 270) (size 1.325 1.8) (layers "B.Cu" "B.Paste" "B.Mask") (roundrect_rratio 0.1886792453)
       (net 1 "GND") (pintype "passive"))
-    (pad "2" smd roundrect (at 1.5625 0 270) (size 1.325 1.8) (layers "B.Cu" "B.Paste" "B.Mask") (roundrect_rratio 0.188679)
+    (pad "2" smd roundrect (at 1.5625 0 270) (size 1.325 1.8) (layers "B.Cu" "B.Paste" "B.Mask") (roundrect_rratio 0.1886792453)
       (net 4 "Net-(LCDScreen1-VOUT)") (pintype "passive"))
     (model "${KICAD6_3DMODEL_DIR}/Capacitor_SMD.3dshapes/C_1206_3216Metric.wrl"
