File: hardware/LCD Module/LCD Module/LCD Module.kicad_sch (KiCad schematic)
At the start: 11 parts, among them J1 Conn_02x04_Counter_Clockwise

Commit message: Working on v2 of HW
Parts:
- J1: value Conn_02x04_Counter_Clockwise -> LCD Screen Connector
Changed lines of the file:
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@@
     (stroke (width 0) (type default))
   )
-  (image (at 275.59 80.01) (scale 0.72312)
+  (image (at 238.76 64.77) (scale 0.72312)
     (data
       iVBORw0KGgoAAAANSUhEUgAABCIAAAXsCAIAAAB8Jr90AAAAA3NCSVQICAjb4U/gAAAACXBIWXMA
@@
       (effects (font (size 1.27 1.27)))
     )
-    (property "Value" "Conn_02x04_Counter_Clockwise" (at 181.61 99.06 0)
+    (property "Value" "LCD Screen Connector" (at 181.61 99.06 0)
       (effects (font (size 1.27 1.27)))
     )
