File: hardware/Bridge System On Ramp.kicad_pcb (KiCad board)
At the start: 2 copper layers, 130.8 x 130.5 mm, 75 parts, among them IC1 SGTL5000XNLA3R2, IC2 AP7313-18SRG-7, U1 Teensy4.1, U2 PEC11R-4015K-N0024

Commit message: Starting to work on Rev 2 of the HW
Parts:
- renumbered ClockStart1 to ClockPlayPause
Connections:
- ClockPlayPause pad 1: GND -> unconnected-(ClockStart1-Pad1)
- ClockPlayPause pad 3: GND -> unconnected-(ClockStart1-Pad3)
- ClockPlayPause pad 4: clockSTART -> GND
- S1 pad 1: GND -> unconnected-(S1-Pad1)
- S1 pad 3: GND -> unconnected-(S1-Pad3)
- S1 pad 4: Button -> GND
Other:
- board text added: "Play/Pause"
- board text removed: "start/stop"
Changed lines of the file:
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@@
   (net 121 "Net-(out1-S)")
   (net 122 "Net-(out2-S)")
+  (net 123 "unconnected-(ClockStart1-Pad1)")
+  (net 124 "unconnected-(ClockStart1-Pad3)")
+  (net 125 "unconnected-(S1-Pad1)")
+  (net 126 "unconnected-(S1-Pad3)")
   (footprint "Alpha potentiometer eurorack:EVUFXL" (layer "F.Cu")
     (at 97.1 38.1)
@@
       (stroke (width 0.2) (type solid)) (layer "F.Fab"))
     (pad "1" thru_hole circle (at 0 -0.031) (size 1.6 1.6) (drill 1.05) (layers "*.Cu" "*.Mask")
-      (net 97 "GND") (pinfunction "1") (pintype "passive"))
+      (net 125 "unconnected-(S1-Pad1)") (pinfunction "1") (pintype "passive"))
     (pad "2" thru_hole circle (at -6.5 -0.031) (size 1.6 1.6) (drill 1.05) (layers "*.Cu" "*.Mask")
       (net 5 "Button") (pinfunction "2") (pintype "passive"))
     (pad "3" thru_hole circle (at 0 -4.531) (size 1.6 1.6) (drill 1.05) (layers "*.Cu" "*.Mask")
-      (net 97 "GND") (pinfunction "3") (pintype "passive"))
+      (net 126 "unconnected-(S1-Pad3)") (pinfunction "3") (pintype "passive"))
     (pad "4" thru_hole circle (at -6.5 -4.531) (size 1.6 1.6) (drill 1.05) (layers "*.Cu" "*.Mask")
-      (net 5 "Button") (pinfunction "4") (pintype "passive"))
+      (net 97 "GND") (pinfunction "4") (pintype "passive"))
     (model "B3W-1000.stp"
       (offset (xyz 0 0 0))
@@
     (property "ki_description" "OMRON ELECTRONIC COMPONENTS - B3W-1000 - SWITCH, SPST-NO, 0.05A, 24VDC, THT")
     (attr through_hole)
-    (fp_text reference "ClockStart1" (at -3.116 -2.281) (layer "F.SilkS")
+    (fp_text reference "ClockPlayPause" (at -3.116 -2.281) (layer "F.SilkS")
         (effects (font (size 1.27 1.27) (thickness 0.254)))
     )
@@
       (stroke (width 0.2) (type solid)) (layer "F.Fab"))
     (pad "1" thru_hole circle (at 0 -0.031) (size 1.6 1.6) (drill 1.05) (layers "*.Cu" "*.Mask")
-      (net 97 "GND") (pinfunction "1") (pintype "passive"))
+      (net 123 "unconnected-(ClockStart1-Pad1)") (pinfunction "1") (pintype "passive"))
     (pad "2" thru_hole circle (at -6.5 -0.031) (size 1.6 1.6) (drill 1.05) (layers "*.Cu" "*.Mask")
       (net 4 "clockSTART") (pinfunction "2") (pintype "passive"))
     (pad "3" thru_hole circle (at 0 -4.531) (size 1.6 1.6) (drill 1.05) (layers "*.Cu" "*.Mask")
-      (net 97 "GND") (pinfunction "3") (pintype "passive"))
+      (net 124 "unconnected-(ClockStart1-Pad3)") (pinfunction "3") (pintype "passive"))
     (pad "4" thru_hole circle (at -6.5 -4.531) (size 1.6 1.6) (drill 1.05) (layers "*.Cu" "*.Mask")
-      (net 4 "clockSTART") (pinfunction "4") (pintype "passive"))
+      (net 97 "GND") (pinfunction "4") (pintype "passive"))
     (model "B3W-1000.stp"
       (offset (xyz 0 0 0))
@@
     )
   )
-  (gr_text "start/stop" (at 154.673654 44.605966) (layer "F.SilkS")
+  (gr_text "Play/Pause" (at 154.673654 44.605966) (layer "F.SilkS")
     (effects (font (size 1 1) (thickness 0.15)) (justify left bottom))
   )

Commit message: Working on v2 of HW
Parts:
- removed BLCK1, CS1, DIN1, DOUT1, LRCLCK1, MCLK1, MISO1, MOSI1, RS1, SCL1, SDA1, reset1: ~, Jumper:SolderJumper-2_P1.3mm_Bridged_Pad1.0x1.5mm
- removed C1: 0.15uF, Capacitor_SMD:C_1206_3216Metric_Pad1.33x1.80mm_HandSolder
- removed C10, C13, C14: 2.2uF, Capacitor_SMD:C_1206_3216Metric_Pad1.33x1.80mm_HandSolder
- removed C11, C12, C15, C16: 0.1uF, Capacitor_SMD:C_1206_3216Metric_Pad1.33x1.80mm_HandSolder
- removed C17, C18: 0uF, Capacitor_SMD:C_1206_3216Metric_Pad1.33x1.80mm_HandSolder
- removed C2, C3, C4, C5, C6, C7, C8, C9: 1uF, Capacitor_SMD:C_1206_3216Metric_Pad1.33x1.80mm_HandSolder
- removed IC1: SGTL5000XNLA3R2, SGTL5000XNLA3R2 Audio Codec Eurorack:QFN40P300X300X60-21N
- removed IC2: AP7313-18SRG-7, AP7313-18SRG-7:SOT96P240X135-3N
- removed LCDScreen1: NHD-C12832A1Z-FSW-FBW-3V3, NHD C12832A1Z FSW LCD SPI Eurorack:NHDC12832A1ZFSWFBW3V3
- added J1: LCD Screen Connector, Connector_PinSocket_2.00mm:PinSocket_2x04_P2.00mm_Vertical_SMD, F.Cu at (207.7, 115.5)
- added J2: Audio Connector, Connector_PinSocket_2.00mm:PinSocket_2x08_P2.00mm_Vertical_SMD, B.Cu at (123.8, 19.1)
- added LED_AttackIN1: LED, LED_THT:LED_D3.0mm, F.Cu at (163.7, 3.69)
- added LED_DecayIN1: LED, LED_THT:LED_D3.0mm, F.Cu at (199.1, 4.07)
- added LED_FilterIN1: LED, LED_THT:LED_D3.0mm, F.Cu at (114.5, 4.20)
- added LED_SeqIN1: LED, LED_THT:LED_D3.0mm, F.Cu at (172.3, 111.7)
- added LED_ShaperIN1: LED, LED_THT:LED_D3.0mm, F.Cu at (64.2, 4.58)
- added LED_WaveformIN1: LED, LED_THT:LED_D3.0mm, F.Cu at (14.0, 4.89)
- added Mult_A_1: PJ301M-12, Thonkiconn:PJ301M-12, F.Cu at (38.2, 40.0)
- added Mult_A_2: PJ301M-12, Thonkiconn:PJ301M-12, F.Cu at (60.4, 39.6)
- added Mult_A_3: PJ301M-12, Thonkiconn:PJ301M-12, F.Cu at (80.7, 39.6)
- added Mult_B_1: PJ301M-12, Thonkiconn:PJ301M-12, F.Cu at (38.3, 56.6)
- added Mult_B_2: PJ301M-12, Thonkiconn:PJ301M-12, F.Cu at (60.5, 56.7)
- added Mult_B_3: PJ301M-12, Thonkiconn:PJ301M-12, F.Cu at (80.6, 56.7)
- added R10: 330, Resistor_SMD:R_1206_3216Metric_Pad1.30x1.75mm_HandSolder, B.Cu at (20.3, 5.08)
- added R11: 330, Resistor_SMD:R_1206_3216Metric_Pad1.30x1.75mm_HandSolder, B.Cu at (178.8, 111.8)
- added R7: 330, Resistor_SMD:R_1206_3216Metric_Pad1.30x1.75mm_HandSolder, B.Cu at (71.6, 4.81)
- added R8: 330, Resistor_SMD:R_1206_3216Metric_Pad1.30x1.75mm_HandSolder, B.Cu at (121.9, 3.95)
- added R9: 330, Resistor_SMD:R_1206_3216Metric_Pad1.30x1.75mm_HandSolder, B.Cu at (171.1, 3.61)
- R1: value 100 -> 330
- Trigger1: renamed from S1; value B3W-1000 -> Adafruit 3488; footprint B3W1050:B3W1050 -> Connector_PinHeader_1.00mm:PinHeader_1x02_P1.00mm_Vertical
- seqIN1: renamed from Clock Out1
- moved R1 163.4 mm to (205.7, 3.53)
- moved U2 141.4 mm to (33.7, 139.6)
- moved ClockPlay1 139.3 mm to (39.3, 108.3)
- moved ClockLED1 138.2 mm to (34.8, 91.4), turned to 0 degrees
- moved EnvDecay1 132.2 mm to (192.4, -27.0)
- moved R6 120.2 mm to (45.7, 89.9), turned to 0 degrees
- moved LFO Out1 101.7 mm to (221.0, 33.5)
- moved EnvAttack1 98.2 mm to (158.6, -27.5)
- moved Decay IN1 97.2 mm to (189.8, 4.11)
- moved OscWaveform1 94.1 mm to (9.02, -27.2)
- moved LFOAmount1 88.4 mm to (184.7, 49.8)
- moved LineIn_L1 86.4 mm to (-1.73, 40.0), turned to 90 degrees
- moved Filter1 85.4 mm to (108.6, -27.2)
- moved Waveform IN1 84.2 mm to (5.07, 4.85), turned to 90 degrees
- moved Shaper1 83.9 mm to (58.8, -27.1)
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- renumbered ClockPlayPause to ClockPlay1
Connections:
- net clockOUT renamed seqIN
- net clockSTART renamed clockPLAY
- Attack IN1 pad 2: unconnected-(Attack IN1-Pad2) -> GND
- Decay IN1 pad 2: unconnected-(Decay IN1-Pad2) -> GND
- Filter IN1 pad 2: unconnected-(Filter IN1-Pad2) -> GND
- LineIn_L1 pad 3: Net-(C17-Pad2) -> Linein_L
- LineIn_R1 pad 3: Net-(C18-Pad1) -> Linein_R
- R1 pad 2: MCLK -> decayIN
- Shaper IN1 pad 2: unconnected-(Shaper IN1-Pad2) -> GND
- Trigger1 pad 1: unconnected-(S1-Pad1) -> Trigger
- Trigger1 pad 2: Button -> GND
- U1 pad 10: Net-(DOUT1-B) -> DOUT
- U1 pad 25: Net-(MCLK1-A) -> unconnected-(U1-33_MCLK2-Pad25)
- U1 pad 4: Button -> Trigger
- U1 pad 40: Net-(SDA1-A) -> SDA
- U1 pad 41: Net-(SCL1-A) -> SCL
- U1 pad 42: Net-(LRCLCK1-A) -> LRCLCK
- U1 pad 43: Net-(BLCK1-A) -> BLCK
- U1 pad 45: LFOAmount -> MCLK
- U1 pad 9: Net-(DIN1-B) -> DIN
- Waveform IN1 pad 2: unconnected-(Waveform IN1-Pad2) -> GND
- out1 pad 3: Net-(IC1-HP_L) -> Headphones_L
- out2 pad 3: Net-(IC1-HP_R) -> Headphones_R
- seqIN1 pad 2: unconnected-(Clock Out1-Pad2) -> GND
Routing:
- net +3.3V: track 433.7 -> 0.00 mm, vias 1 -> 0
- net LFORate: track 129.0 -> 0.00 mm, vias 2 -> 0
- net LFOWave: track 123.5 -> 0.00 mm, vias 1 -> 0
- net OscWaveform: track 115.7 -> 0.00 mm
- net filterIN: track 114.5 -> 0.00 mm, vias 1 -> 0
- net seqIN: track 114.0 -> 0.00 mm
- net shaperIN: track 113.7 -> 0.00 mm, vias 1 -> 0
- net Filter: track 112.9 -> 0.00 mm, vias 1 -> 0
- net LFOAmount: track 112.9 -> 0.00 mm
- net Shaper: track 111.2 -> 0.00 mm
- net waveformIN: track 103.9 -> 0.00 mm, vias 1 -> 0
- net attackIN: track 92.6 -> 0.00 mm, vias 1 -> 0
- net Net-(IC1-HP_L): track 91.8 -> 0.00 mm, vias 1 -> 0
- net Net-(IC1-HP_R): track 90.5 -> 0.00 mm, vias 1 -> 0
- net seq1LED: track 84.9 -> 0.00 mm
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Other:
- board size 130.8 x 130.5 mm -> 266.4 x 221.8 mm
- board text added: "2023 v2"
- board text added: "AMOUNT"
- board text added: "ATTACK"
- board text added: "AUDIO INPUT"
- board text added: "BRIDGE SYSTEM"
- board text added: "CLEAN"
- board text added: "CLOCK"
- board text added: "CLOCK RATE"
- board text added: "CRUSHED"
- board text added: "CUTOFF"
- board text added: "DECAY"
- board text added: "DISTORT"
- board text added: "ENVELOPE"
- board text added: "FAST"
- board text added: "FILTER"
- board text added: "HIGHPASS"
- board text added: "INV MOD OUT"
- board text added: "JLCJLCJLCJLC"
- board text added: "LOWPASS"
- board text added: "MOD OUT"
- board text added: "MODULATION"
- board text added: "MULT"
- board text added: "ONRAMP"
- board text added: "OSCILLATOR"
- board text added: "OUT A"
- board text added: "OUT B"
- board text added: "OUTPUT"
- board text added: "OUTPUT 1"
- board text added: "OUTPUT 2"
- board text added: "RATE"
- board text added: "SEQ OUT"
- board text added: "SEQUENCER"
- board text added: "SLOW"
- board text added: "TRIGGER"
- board text added: "TRIGGER OUT"
- board text added: "WAVEFORM"
- board text removed: "Bridge System: On Ramp v1 2023"
- board text removed: "North Coast Modular Collective"
- board text removed: "Play/Pause"
- board text removed: "Stereo"
- board text removed: "output"

Commit message: mostly hardware updates - also MUX chip test code
Parts:
- Trigger1: footprint Connector_PinHeader_1.00mm:PinHeader_1x02_P1.00mm_Vertical -> Connector_PinSocket_2.54mm:PinSocket_1x02_P2.54mm_Horizontal
Connections:
- R1 pad 2: decayIN -> Net-(decayIN1-B)
- R10 pad 2: waveformIN -> Net-(waveformIN1-B)
- R11 pad 2: seqIN -> Net-(seqIN2-B)
- R7 pad 2: shaperIN -> Net-(shaperIN1-B)
- R8 pad 2: filterIN -> Net-(filterIN1-B)
- R9 pad 2: attackIN -> Net-(attackIN1-B)
Routing:
- net (no net): vias 8 -> 0
Other:
- outline, holes or cut-outs redrawn
- board text added: "1 U = 44.45 mm (raw) 3U = 133.4 mm (raw) or 128.5 mm at Doepfer spec (for rail rims and vertical space between rows)"
- board text added: "2023 v3"
- board text removed: "2023 v2"
