File: hardware/Bridge System On Ramp.kicad_sch (KiCad schematic)
At the start: 75 parts, among them IC1 SGTL5000XNLA3R2, IC2 AP7313-18SRG-7, U1 Teensy4.1, U2 PEC11R-4015K-N0024

Commit message: Starting to work on Rev 2 of the HW
Connections:
- net Button: no longer S1.4
- net GND: now also ClockStart1.4, S1.4; no longer ClockStart1.1, ClockStart1.3, S1.1, S1.3
- net clockSTART renamed clockPLAY
- net clockPLAY: no longer ClockStart1.4
Other:
- note added: "Needed Changes: 1) [DONE] fix the button wiring 2) rewire the outputs to be L/R mirrors, not L then R 3) Add standoff holes with space around edges to mount it in a box if needed 4) [DONE] Rename clock start-stop to clock play-pause 5) Swap "trigger" button with arcade button in schematic/PCB 6) Add LEDs to the inputs to show patched signal values 7) For the patch out jacks, make it so the output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"
- note removed: "Needed Changes: 1) fix the button wiring 2) rewire the outputs to be L/R mirrors, not L then R 3) Add standoff holes with space around edges to mount it in a box if needed 4) Rename clock start-stop to clock play-pause 5) Swap "trigger" button with arcade button in schematic/PCB 6) Add LEDs to the inputs to show patched signal values 7) For the patch out jacks, make it so the output/input doesn't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"
Changed lines of the file:
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@@
   (title_block
     (title "Bridge System: On Ramp")
-    (date "2023-05-09")
-    (rev "1")
+    (date "2023-11-12")
+    (rev "2")
     (company "North Coast Modular Collective")
     (comment 1 "www.northcoastmodularcollective.com")
@@
   (junction (at 31.75 238.76) (diameter 0) (color 0 0 0 0)
   )
-  (junction (at 247.65 44.45) (diameter 0) (color 0 0 0 0)
-  )
   (junction (at 52.07 176.53) (diameter 0) (color 0 0 0 0)
   )
@@
   (junction (at 36.83 142.24) (diameter 0) (color 0 0 0 0)
   )
-  (junction (at 266.7 26.67) (diameter 0) (color 0 0 0 0)
-  )
   (junction (at 43.18 142.24) (diameter 0) (color 0 0 0 0)
   )
-  (junction (at 267.97 41.91) (diameter 0) (color 0 0 0 0)
-  )
   (junction (at 222.25 99.06) (diameter 0) (color 0 0 0 0)
   )
   (junction (at 52.07 142.24) (diameter 0) (color 0 0 0 0)
   )
-  (junction (at 267.97 44.45) (diameter 0) (color 0 0 0 0)
-  )
   (junction (at 222.25 116.84) (diameter 0) (color 0 0 0 0)
   )
-  (junction (at 246.38 26.67) (diameter 0) (color 0 0 0 0)
-  )
   (junction (at 66.04 190.5) (diameter 0) (color 0 0 0 0)
   )
-  (junction (at 266.7 24.13) (diameter 0) (color 0 0 0 0)
-  )
   (junction (at 121.92 220.98) (diameter 0) (color 0 0 0 0)
   )
@@
     (stroke (width 0) (type default))
   )
-  (wire (pts (xy 267.97 44.45) (xy 271.78 44.45))
-    (stroke (width 0) (type default))
-  )
   (wire (pts (xy 243.84 236.22) (xy 246.38 236.22))
     (stroke (width 0) (type default))
@@
     (stroke (width 0) (type default))
   )
-  (wire (pts (xy 247.65 41.91) (xy 247.65 44.45))
-    (stroke (width 0) (type default))
-  )
   (wire (pts (xy 247.65 129.54) (xy 248.92 129.54))
     (stroke (width 0) (type default))
@@
     (stroke (width 0) (type default))
   )
-  (wire (pts (xy 271.78 44.45) (xy 271.78 48.26))
-    (stroke (width 0) (type default))
-  )
   (wire (pts (xy 95.25 213.36) (xy 99.06 213.36))
     (stroke (width 0) (type default))
@@
     (stroke (width 0) (type default))
   )
-  (wire (pts (xy 270.51 26.67) (xy 270.51 30.48))
-    (stroke (width 0) (type default))
-  )
   (wire (pts (xy 180.34 223.52) (xy 180.34 226.06))
     (stroke (width 0) (type default))
@@
     (stroke (width 0) (type default))
   )
-  (wire (pts (xy 267.97 40.64) (xy 267.97 41.91))
-    (stroke (width 0) (type default))
-  )
-  (wire (pts (xy 246.38 24.13) (xy 246.38 26.67))
-    (stroke (width 0) (type default))
-  )
   (wire (pts (xy 102.87 46.99) (xy 106.68 46.99))
     (stroke (width 0) (type default))
@@
     (stroke (width 0) (type default))
   )
-  (wire (pts (xy 266.7 24.13) (xy 266.7 26.67))
-    (stroke (width 0) (type default))
-  )
-  (wire (pts (xy 266.7 26.67) (xy 270.51 26.67))
+  (wire (pts (xy 245.11 41.91) (xy 247.65 41.91))
     (stroke (width 0) (type default))
   )
@@
     (stroke (width 0) (type default))
   )
-  (wire (pts (xy 266.7 22.86) (xy 266.7 24.13))
-    (stroke (width 0) (type default))
-  )
   (wire (pts (xy 66.04 190.5) (xy 69.85 190.5))
     (stroke (width 0) (type default))
@@
     (stroke (width 0) (type default))
   )
+  (wire (pts (xy 243.84 24.13) (xy 246.38 24.13))
+    (stroke (width 0) (type default))
+  )
   (wire (pts (xy 238.76 127) (xy 240.03 127))
     (stroke (width 0) (type default))
@@
     (stroke (width 0) (type default))
   )
-  (wire (pts (xy 267.97 41.91) (xy 267.97 44.45))
-    (stroke (width 0) (type default))
-  )
   (wire (pts (xy 165.1 224.79) (xy 165.1 227.33))
     (stroke (width 0) (type default))
@@
     (effects (font (size 1.27 1.27)) (justify left bottom))
   )
-  (text "Needed Changes:\n1) fix the button wiring\n2) rewire the outputs to be L/R mirrors, not L then R\n3) Add standoff holes with space around edges to mount it in a box if needed\n4) Rename clock start-stop to clock play-pause\n5) Swap \"trigger\" button with arcade button in schematic/PCB\n6) Add LEDs to the inputs to show patched signal values\n7) For the patch out jacks, make it so the output/input doesn't need a pullup resistor?\n8) Rev 3: Make input jacks able to handle Euro level inputs - Use op amps?\n\n"
+  (text "Needed Changes:\n1) [DONE] fix the button wiring\n2) rewire the outputs to be L/R mirrors, not L then R\n3) Add standoff holes with space around edges to mount it in a box if needed\n4) [DONE] Rename clock start-stop to clock play-pause\n5) Swap \"trigger\" button with arcade button in schematic/PCB\n6) Add LEDs to the inputs to show patched signal values\n7) For the patch out jacks, make it so the output/input doesn't need a pullup resistor?\n8) Rev 3: Make input jacks able to handle Euro level inputs - Use op amps?\n9) MCLK from Audio board is supposed to go to pin 23 not 33. Currently LFO ammount is at 23, need to find a new home for it.\n10) Look into a MUX for analog pins, like this one: CD74HC4051-EP Analog Multiplexer and Demultiplexer \n11) Reorganize the parts on the PCB to match relative positions of new layout design\n"
     (at 104.14 330.2 0)
     (effects (font (size 2 2)) (justify left bottom))
@@
     )
   )
-  (global_label "clockSTART" (shape input) (at 241.3 44.45 180) (fields_autoplaced)
+  (global_label "clockPLAY" (shape input) (at 241.3 44.45 180) (fields_autoplaced)
     (effects (font (size 1.27 1.27)) (justify right))
-    (property "Intersheetrefs" "${INTERSHEET_REFS}" (at 227.8714 44.45 0)
+    (property "Intersheetrefs" "${INTERSHEET_REFS}" (at 228.8994 44.45 0)
       (effects (font (size 1.27 1.27)) (justify right) hide)
     )
@@
     )
   )
-  (global_label "clockSTART" (shape input) (at 95.25 90.17 0) (fields_autoplaced)
+  (global_label "clockPLAY" (shape input) (at 95.25 90.17 0) (fields_autoplaced)
     (effects (font (size 1.27 1.27)) (justify left))
-    (property "Intersheetrefs" "${INTERSHEET_REFS}" (at 108.6786 90.17 0)
+    (property "Intersheetrefs" "${INTERSHEET_REFS}" (at 107.6506 90.17 0)
       (effects (font (size 1.27 1.27)) (justify left) hide)
     )
@@
     )
   )
-  (symbol (lib_id "power:GND") (at 271.78 48.26 0) (unit 1)
+  (symbol (lib_id "power:GND") (at 245.11 41.91 270) (unit 1)
     (in_bom yes) (on_board yes) (dnp no)
-    (property "Reference" "#PWR036" (at 271.78 54.61 0)
+    (property "Reference" "#PWR036" (at 238.76 41.91 0)
       (effects (font (size 1.27 1.27)) hide)
     )
-    (property "Value" "GND" (at 271.78 52.07 0)
+    (property "Value" "GND" (at 241.3 41.91 0)
       (effects (font (size 1.27 1.27)))
     )
-    (property "Footprint" "" (at 271.78 48.26 0)
+    (property "Footprint" "" (at 245.11 41.91 0)
       (effects (font (size 1.27 1.27)) hide)
     )
-    (property "Datasheet" "" (at 271.78 48.26 0)
+    (property "Datasheet" "" (at 245.11 41.91 0)
       (effects (font (size 1.27 1.27)) hide)
     )
@@
     )
   )
-  (symbol (lib_id "power:GND") (at 270.51 30.48 0) (unit 1)
+  (symbol (lib_id "power:GND") (at 243.84 24.13 270) (unit 1)
     (in_bom yes) (on_board yes) (dnp no)
-    (property "Reference" "#PWR09" (at 270.51 36.83 0)
+    (property "Reference" "#PWR09" (at 237.49 24.13 0)
       (effects (font (size 1.27 1.27)) hide)
     )
-    (property "Value" "GND" (at 270.51 34.29 0)
+    (property "Value" "GND" (at 240.03 24.13 0)
       (effects (font (size 1.27 1.27)))
     )
-    (property "Footprint" "" (at 270.51 30.48 0)
+    (property "Footprint" "" (at 243.84 24.13 0)
       (effects (font (size 1.27 1.27)) hide)
     )
-    (property "Datasheet" "" (at 270.51 30.48 0)
+    (property "Datasheet" "" (at 243.84 24.13 0)
       (effects (font (size 1.27 1.27)) hide)
     )

Commit message: Working on v2 of HW
Parts:
- removed BLCK1, CS1, DIN1, DOUT1, LRCLCK1, MCLK1, MISO1, MOSI1, RS1, SCL1, SDA1, reset1: ~, Jumper:SolderJumper-2_P1.3mm_Bridged_Pad1.0x1.5mm, symbol Jumper:SolderJumper_2_Bridged
- removed C1: 0.15uF, Capacitor_SMD:C_1206_3216Metric_Pad1.33x1.80mm_HandSolder, symbol Device:C
- removed C10, C13, C14: 2.2uF, Capacitor_SMD:C_1206_3216Metric_Pad1.33x1.80mm_HandSolder, symbol Device:C
- removed C11, C12, C15, C16: 0.1uF, Capacitor_SMD:C_1206_3216Metric_Pad1.33x1.80mm_HandSolder, symbol Device:C
- removed C17, C18: 0uF, Capacitor_SMD:C_1206_3216Metric_Pad1.33x1.80mm_HandSolder, symbol Device:C
- removed C2, C3, C4, C5, C6, C7, C8, C9: 1uF, Capacitor_SMD:C_1206_3216Metric_Pad1.33x1.80mm_HandSolder, symbol Device:C
- removed IC1: SGTL5000XNLA3R2, SGTL5000XNLA3R2 Audio Codec Eurorack:QFN40P300X300X60-21N, symbol SGTL5000XNLA3R2:SGTL5000XNLA3R2
- removed IC2: AP7313-18SRG-7, AP7313-18SRG-7:SOT96P240X135-3N, symbol AP7313-18SRG-7:AP7313-18SRG-7
- removed LCDScreen1: NHD-C12832A1Z-FSW-FBW-3V3, NHD C12832A1Z FSW LCD SPI Eurorack:NHDC12832A1ZFSWFBW3V3, symbol NHD-C12832A1Z-FSW-FBW-3V3:NHD-C12832A1Z-FSW-FBW-3V3
- added J1: LCD Screen Connector, Connector_PinSocket_2.00mm:PinSocket_2x04_P2.00mm_Vertical_SMD, symbol Audio Module Eurorack:Conn_02x04_Counter_Clockwise
- added J2: Audio Connector, Connector_PinSocket_2.00mm:PinSocket_2x08_P2.00mm_Vertical_SMD, symbol PCM_4ms_Connector:Conn_02x08
- added LED_AttackIN, LED_DecayIN, LED_FilterIN, LED_SeqIN, LED_ShaperIN, LED_WaveformIN: LED, LED_THT:LED_D3.0mm, symbol Device:LED
- added Mult_A_1, Mult_A_2, Mult_A_3, Mult_B_1, Mult_B_2, Mult_B_3: PJ301M-12, Thonkiconn:PJ301M-12, symbol thonkiconn:PJ301M-12
- added R10, R11, R7, R8, R9: 330, Resistor_SMD:R_1206_3216Metric_Pad1.30x1.75mm_HandSolder, symbol Device:R_US
- R1: value 100 -> 330
- Trigger1: renamed from S1; value B3W-1000 -> Adafruit 3488; footprint B3W1050 -> Connector_PinHeader_1.00mm:PinHeader_1x02_P1.00mm_Vertical; symbol B3W-1000:B3W-1000 -> Switch:SW_Push
- seqIN1: renamed from Clock Out1
- renumbered ClockStart1 to ClockPlay1
Connections:
- net +3.3V: now also J1.1 (Pin_1), J1.3 (Pin_3), J2.2 (P2)
- net BLCK: now also U1.43 (21_A7_RX5_BCLK1), J2.15 (-12V)
- net CS1: now also J1.2 (Pin_2)
- net DIN: now also U1.9 (7_RX2_OUT1A), J2.13 (-12)
- net DOUT: now also U1.10 (8_TX2_IN1), J2.11 (GND)
- net GND: now also Attack IN1.2, Decay IN1.2, Filter IN1.2, Shaper IN1.2, Trigger1.2, Waveform IN1.2, seqIN1.2, J1.8 (Pin_8), J2.1 (P1), LED_AttackIN.1 (K), LED_DecayIN.1 (K), LED_FilterIN.1 (K), LED_SeqIN.1 (K), LED_ShaperIN.1 (K), LED_WaveformIN.1 (K); no longer Trigger1.4
- net LFOAmount: no longer U1.45 (23_A9_CRX1_MCLK1)
- net LRCLCK: now also U1.42 (20_A6_TX5_LRCLK1), J2.9 (GND)
- net MCLK: now also U1.45 (23_A9_CRX1_MCLK1), J2.7 (12V); no longer R1.2
- net MISO: now also J1.4 (Pin_4)
- net MOSI: now also J1.7 (Pin_7)
- net RS: now also J1.6 (Pin_6)
- net SCL: now also U1.41 (19_A5_SCL), J2.5 (+12V)
- net SDA: now also U1.40 (18_A4_SDA), J2.3 (P3)
- net attackIN: now also R9.2
- net decayIN: now also R1.2
- net filterIN: now also R8.2
- net reset: now also J1.5 (Pin_5)
- net shaperIN: now also R7.2
- net waveformIN: now also R10.2
- net Linein_R: now reaches LineIn_R1.3
- net Linein_R: now also J2.10 (GND)
- net Headphones_R: now reaches out2.3 (E)
- net Headphones_R: now also J2.6 (P6)
- net Trigger: now reaches Trigger1.1
- net Trigger: now also U1.4 (2_OUT2)
- net Headphones_L: now reaches out1.3 (E)
- net Headphones_L: now also J2.4 (P4)
- net at R1.1: now also LED_DecayIN.2 (A)
- net Linein_L: now reaches LineIn_L1.3
- net Linein_L: now also J2.8 (+12V)
- removed net Button: Trigger1.2, U1.4 (2_OUT2)
- net clockOUT renamed seqIN
- net seqIN: now also R11.2
- new net: Mult_A_1.1, Mult_A_2.1, Mult_A_3.1
- new net: Mult_A_1.3, Mult_A_2.3, Mult_A_3.3
- new net: LED_ShaperIN.2 (A), R7.1
- new net: LED_WaveformIN.2 (A), R10.1
- new net: LED_FilterIN.2 (A), R8.1
- new net: Mult_B_1.1, Mult_B_2.1, Mult_B_3.1
- new net: Mult_B_1.3, Mult_B_2.3, Mult_B_3.3
- new net: LED_SeqIN.2 (A), R11.1
- new net: LED_AttackIN.2 (A), R9.1
- new net Lineout_L: J2.14 (-12V)
- new net Lineout_R: J2.16 (P16)
- new net Mic: J2.12 (GND)
Other:
- note added: "Change Log: 1) [DONE] fix the button wiring 2) rewire the outputs to be L/R mirrors, not L then R 3) Add standoff holes with space around edges to mount it in a box if needed 4) [DONE] Rename clock start-stop to clock play-pause 5) [DONE] Swap "trigger" button with arcade button in schematic/PCB 6) Add LEDs to the inputs to show patched signal values 7) For the patch out jacks, make it so the out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"
- note removed: "MCLK 23 (MCLK1) Audio Audio Master Clock, 11.29 MHz BCLK 21 (BCLK1) Audio Audio Bit Clock, 1.41 or 2.82 MHz LRCLK 20(LRCLK1) Audio Audio Left/Right Clock, 44.1 kHz DIN 7(OUT1A) Audio Output Audio Data from Teensy to Audio Shield Goes to both headphone jack and Line-Out pins DOUT 8 (IN1) Audio Input Audio Data from Audio Shield to Teensy Comes from either Microphone or Line-In pins SCL 19 Audio Co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"
- note removed: "Needed Changes: 1) [DONE] fix the button wiring 2) rewire the outputs to be L/R mirrors, not L then R 3) Add standoff holes with space around edges to mount it in a box if needed 4) [DONE] Rename clock start-stop to clock play-pause 5) Swap "trigger" button with arcade button in schematic/PCB 6) Add LEDs to the inputs to show patched signal values 7) For the patch out jacks, make it so the output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"
- note removed: "creates 1.8v for VDDD"
- note removed: "creates a more filtered version of 3.3v"
- moved on the sheet: EnvAttack1, EnvDecay1, Filter1, LFOAmount1, LFORate1, LFOWave1, LineIn_L1, LineIn_R1, OscWaveform1, R2, R3, R4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

Commit message: mostly hardware updates - also MUX chip test code
Parts:
- added attackIN1, decayIN1, filterIN1, seqIN2, shaperIN1, waveformIN1: ~, symbol Jumper:SolderJumper_2_Bridged
- Trigger1: footprint Connector_PinHeader_1.00mm:PinHeader_1x02_P1.00mm_Vertical -> Connector_PinSocket_2.54mm:PinSocket_1x02_P2.54mm_Horizontal
- renumbered LED_AttackIN to LED_AttackIN1, LED_DecayIN to LED_DecayIN1, LED_FilterIN to LED_FilterIN1, LED_SeqIN to LED_SeqIN1, LED_ShaperIN to LED_ShaperIN1, LED_WaveformIN to LED_WaveformIN1
Connections:
- net attackIN: now also attackIN1.1 (A); no longer R9.2
- net decayIN: now also decayIN1.1 (A); no longer R1.2
- net filterIN: now also filterIN1.1 (A); no longer R8.2
- net seqIN: now also seqIN2.1 (A); no longer R11.2
- net shaperIN: now also shaperIN1.1 (A); no longer R7.2
- net waveformIN: now also waveformIN1.1 (A); no longer R10.2
- new net: R7.2, shaperIN1.2 (B)
- new net: R9.2, attackIN1.2 (B)
- new net: R10.2, waveformIN1.2 (B)
- new net: R1.2, decayIN1.2 (B)
- new net: R8.2, filterIN1.2 (B)
- new net: R11.2, seqIN2.2 (B)
Other:
- note added: "Change Log (completed and in which version) [DONE v2] fix the button wiring [DONE v2] Rename clock start-stop to clock play-pause [DONE v2] Swap "trigger" button with arcade button in schematic/PCB [DONE v2] MCLK from Audio board is supposed to go to pin 23 not 33. Currently LFO ammount is at 23, need to find a new home for it. [DONE v2] Reorganize the parts on the PCB to match relative positions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"
- note added: "Could put a clock output here? Op amp to amp to euro?"
- note added: "To-Do list for V3: -rewire the outputs to be L/R mirrors, not L then R (will probably need audio taper and dual pole pots) -Add standoff holes with space around edges to mount it in a box if needed (don't use vias) -Add LEDs to the inputs to show patched signal values -For the patch out jacks, make it so the output/input doesn't need a pullup resistor? (only if using PWM instead of CV) -Make inpu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"
- note removed: "Change Log: 1) [DONE] fix the button wiring 2) rewire the outputs to be L/R mirrors, not L then R 3) Add standoff holes with space around edges to mount it in a box if needed 4) [DONE] Rename clock start-stop to clock play-pause 5) [DONE] Swap "trigger" button with arcade button in schematic/PCB 6) Add LEDs to the inputs to show patched signal values 7) For the patch out jacks, make it so the out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"
- moved on the sheet: ClockLED1, ClockPlay1, J1, J2, LED_AttackIN1, LED_DecayIN1, LED_FilterIN1, LED_SeqIN1, LED_ShaperIN1, LED_WaveformIN1, LFO Out1, LineIn_L1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
